File: vco-4pasos-v-0-2/_restore_backup_2026-10-01T15-18-06-968/vco-4pasos-v-0-2.kicad_sch (KiCad schematic)
At the start: 27 parts, among them J1 Screw_Terminal_01x02, J2 Screw_Terminal_01x04, J3 Screw_Terminal_01x04, U1 HEF4093B

Commit message: actualizacion esquematico
Parts:
- removed C10: 1u, Capacitor_THT:CP_Radial_D4.0mm_P2.00mm, symbol Device:C_Polarized
- removed C11, C9: 0.22, Capacitor_THT:CP_Radial_D4.0mm_P2.00mm, symbol Device:C_Polarized
- removed C12: 0.47u, Capacitor_THT:CP_Radial_D4.0mm_P2.00mm, symbol Device:C_Polarized
- removed C5: 2.2u, Capacitor_THT:CP_Radial_D4.0mm_P2.00mm, symbol Device:C_Polarized
- removed C6: 4.7u, Capacitor_THT:CP_Radial_D4.0mm_P2.00mm, symbol Device:C_Polarized
- removed C7: 3.3u, Capacitor_THT:CP_Radial_D4.0mm_P2.00mm, symbol Device:C_Polarized
- removed C8: 0.1u, Capacitor_THT:CP_Radial_D4.0mm_P2.00mm, symbol Device:C_Polarized
- C1, C4: value 0.22u -> 1u
- C2: value 0.1u -> 1u
- C3: value 0.47u -> 1u
- renumbered C13 to C5
Connections:
- net GND: now also C1.2, C2.2, C4.2
- net at RV2.2, U1.6: now also C2.1; no longer C4.1
- net at RV4.2, U1.13: now also C4.1
- net at RV3.2, U1.9: now also C3.1
