File: vco-4pasos-v-0-3/vco-4pasos-v-0-3.kicad_pcb (KiCad board)
At the start: 2 copper layers, 50 x 50 mm, 19 parts, among them J1 Screw_Terminal_01x02, J2 Screw_Terminal_01x04, J3 Screw_Terminal_01x04, U1 HEF4093B

Commit message: actualizacion esquematico
Parts:
- added C10: 1u, Capacitor_THT:CP_Radial_D4.0mm_P2.00mm, F.Cu at (91.3, 46.3)
- added C11: 0.22, Capacitor_THT:CP_Radial_D4.0mm_P2.00mm, F.Cu at (91.3, 51.8)
- added C12: 0.47u, Capacitor_THT:CP_Radial_D4.0mm_P2.00mm, F.Cu at (91.3, 57.4)
- added C2: 0.1u, Capacitor_THT:CP_Radial_D4.0mm_P2.00mm, F.Cu at (80.1, 46.3)
- added C3: 0.47u, Capacitor_THT:CP_Radial_D4.0mm_P2.00mm, F.Cu at (80.1, 51.8)
- added C4: 0.22u, Capacitor_THT:CP_Radial_D4.0mm_P2.00mm, F.Cu at (80.1, 57.4)
- added C5: 2.2u, Capacitor_THT:CP_Radial_D4.0mm_P2.00mm, F.Cu at (80.1, 62.9)
- added C6: 4.7u, Capacitor_THT:CP_Radial_D4.0mm_P2.00mm, F.Cu at (85.7, 46.3)
- added C7: 3.3u, Capacitor_THT:CP_Radial_D4.0mm_P2.00mm, F.Cu at (85.7, 51.8)
- added C8: 0.1u, Capacitor_THT:CP_Radial_D4.0mm_P2.00mm, F.Cu at (85.7, 57.4)
- added C9: 0.22, Capacitor_THT:CP_Radial_D4.0mm_P2.00mm, F.Cu at (85.7, 62.9)
- C1: value 1u -> 0.22u
- renumbered C5 to C13
Connections:
- C1 pad 2: GND -> Net-(C1-Pad2)
- RV2 pad 2: Net-(C2-Pad1) -> Net-(C4-Pad1)
- RV3 pad 2: Net-(C3-Pad1) -> Net-(C7-Pad1)
- RV4 pad 2: Net-(C4-Pad1) -> Net-(C10-Pad1)
- U1 pad 13: Net-(C4-Pad1) -> Net-(C10-Pad1)
- U1 pad 6: Net-(C2-Pad1) -> Net-(C4-Pad1)
- U1 pad 9: Net-(C3-Pad1) -> Net-(C7-Pad1)
