File: vco-4pasos-v-0-4/vco-4pasos-v-0-4.kicad_sch (KiCad schematic)
At the start: 21 parts, among them J1 Screw_Terminal_01x02, J2 Screw_Terminal_01x04, J3 Screw_Terminal_01x04, U1 HEF4093B

Commit message: agregar pcb
Parts:
- renumbered C3 to C1, C1 to C2, C4 to C3, C8 to C4, C10 to C5, C11 to C6, C13 to C7
Changed lines of the file:
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@@
 		(in_pos_files yes)
 		(dnp no)
-		(property "Reference" "C1"
+		(property "Reference" "C2"
 			(at 55.88 84.2009 0)
 			(show_name no)
@@
 			(project "vco-4pasos-v-0-4"
 				(path "/e3b6b2bd-18d6-4b60-b41d-e2b400c48c4f"
-					(reference "C1")
+					(reference "C2")
 					(unit 1)
 				)
@@
 		(in_pos_files yes)
 		(dnp no)
-		(property "Reference" "C8"
+		(property "Reference" "C4"
 			(at 106.68 84.2009 0)
 			(show_name no)
@@
 			(project "vco-4pasos-v-0-4"
 				(path "/e3b6b2bd-18d6-4b60-b41d-e2b400c48c4f"
-					(reference "C8")
+					(reference "C4")
 					(unit 1)
 				)
@@
 		(dnp no)
 		(fields_autoplaced yes)
-		(property "Reference" "C13"
+		(property "Reference" "C7"
 			(at 195.58 60.9599 0)
 			(show_name no)
@@
 			(project "vco-4pasos-v-0-4"
 				(path "/e3b6b2bd-18d6-4b60-b41d-e2b400c48c4f"
-					(reference "C13")
+					(reference "C7")
 					(unit 1)
 				)
@@
 		(in_pos_files yes)
 		(dnp no)
-		(property "Reference" "C10"
+		(property "Reference" "C5"
 			(at 132.08 90.5509 0)
 			(show_name no)
@@
 			(project "vco-4pasos-v-0-4"
 				(path "/e3b6b2bd-18d6-4b60-b41d-e2b400c48c4f"
-					(reference "C10")
+					(reference "C5")
 					(unit 1)
 				)
@@
 		(in_pos_files yes)
 		(dnp no)
-		(property "Reference" "C4"
+		(property "Reference" "C3"
 			(at 81.28 84.2009 0)
 			(show_name no)
@@
 			(project "vco-4pasos-v-0-4"
 				(path "/e3b6b2bd-18d6-4b60-b41d-e2b400c48c4f"
-					(reference "C4")
+					(reference "C3")
 					(unit 1)
 				)
@@
 		(in_pos_files yes)
 		(dnp no)
-		(property "Reference" "C11"
+		(property "Reference" "C6"
 			(at 144.78 90.5509 0)
 			(show_name no)
@@
 			(project "vco-4pasos-v-0-4"
 				(path "/e3b6b2bd-18d6-4b60-b41d-e2b400c48c4f"
-					(reference "C11")
+					(reference "C6")
 					(unit 1)
 				)
@@
 		(in_pos_files yes)
 		(dnp no)
-		(property "Reference" "C3"
+		(property "Reference" "C1"
 			(at 41.91 84.2009 0)
 			(show_name no)
@@
 			(project "vco-4pasos-v-0-4"
 				(path "/e3b6b2bd-18d6-4b60-b41d-e2b400c48c4f"
-					(reference "C3")
-					(unit 1)
-				)
+					(reference "C1")
+					(unit 1)
+				)
