File: vco-4pasos-v-0-4/vco-4pasos-v-0-4.kicad_pcb (KiCad board)
At the start: 2 copper layers, 50 x 50 mm, 30 parts, among them J1 Screw_Terminal_01x02, J2 Screw_Terminal_01x04, J3 Screw_Terminal_01x04, U1 HEF4093B

Commit message: agregar pcb
Parts:
- removed C10: 1u, Capacitor_THT:CP_Radial_D4.0mm_P2.00mm
- removed C11, C9: 0.22, Capacitor_THT:CP_Radial_D4.0mm_P2.00mm
- removed C12: 0.47u, Capacitor_THT:CP_Radial_D4.0mm_P2.00mm
- removed C13: 100n, Capacitor_THT:C_Disc_D5.0mm_W2.5mm_P2.50mm
- removed the C2 at (80.1, 46.3)
- removed the C2 at (42.0, 45.0)
- removed the C3 at (42.0, 53.0)
- removed the C3 at (80.1, 51.8)
- removed the C4 at (80.1, 57.4)
- removed the C4 at (42.0, 57.0)
- removed C8: 0.1u, Capacitor_THT:CP_Radial_D4.0mm_P2.00mm
- added C2: 0.27u, Capacitor_THT:CP_Radial_D4.0mm_P2.00mm, F.Cu at (46.0, 41.0)
- added C3: 0.22u, Capacitor_THT:CP_Radial_D4.0mm_P2.00mm, F.Cu at (40.0, 50.0)
- added C4: 0.1u, Capacitor_THT:CP_Radial_D4.0mm_P2.00mm, F.Cu at (46.0, 50.0)
- C1: value 0.22u -> 0.33u
- C5: value 2.2u -> 0.22u
- C6: value 4.7u -> 0.47
- C7: value 3.3u -> 100n; footprint Capacitor_THT:CP_Radial_D4.0mm_P2.00mm -> Capacitor_THT:C_Disc_D5.0mm_W2.5mm_P2.50mm
- moved C6 41.7 mm to (46.0, 59.0)
- moved C5 40.3 mm to (40.0, 59.0)
- moved C7 34.5 mm to (53.0, 41.0)
- moved R3 9.57 mm to (52.9, 68.0), turned to 0 degrees
- moved R1 6.01 mm to (52.9, 59.0), turned to 0 degrees
- moved R4 5.68 mm to (62.8, 72.0), turned to 0 degrees
- moved C1 2.83 mm to (40.0, 41.0), turned to 0 degrees
- moved R2 2.65 mm to (62.8, 63.0), turned to 0 degrees
- moved RV1 1.46 mm to (31.0, 34.5)
- moved RV2 1.46 mm to (31.0, 42.5)
- moved RV3 1.46 mm to (31.0, 50.5)
- moved RV4 1.46 mm to (31.0, 58.5)
Connections:
- C1 pad 2: Net-(C1-Pad2) -> GND
- C5 pad 1: Net-(C4-Pad2) -> Net-(C5-Pad1)
- C5 pad 2: Net-(C5-Pad2) -> GND
- C6 pad 1: Net-(C5-Pad2) -> Net-(C5-Pad1)
- C7 pad 1: Net-(C7-Pad1) -> VCC
- C7 pad 2: Net-(C7-Pad2) -> GND
- RV3 pad 2: Net-(C7-Pad1) -> Net-(C4-Pad1)
- RV4 pad 2: Net-(C10-Pad1) -> Net-(C5-Pad1)
- U1 pad 13: Net-(C10-Pad1) -> Net-(C5-Pad1)
- U1 pad 9: Net-(C7-Pad1) -> Net-(C4-Pad1)

Commit message: agregar v-0-4 pcb
Parts:
- moved J3 21.5 mm to (69.0, 69.6), turned to 90 degrees
- moved R2 14.8 mm to (58.0, 49.0), turned to -90 degrees
- moved R1 14.0 mm to (52.9, 45.0), turned to -90 degrees
- moved R4 9.86 mm to (59.0, 62.9), turned to -90 degrees
- moved R3 8.08 mm to (52.9, 59.9), turned to -90 degrees
- moved C4 7.45 mm to (41.0, 55.5), turned to -90 degrees
- moved C6 3.35 mm to (47.5, 62.0), turned to -90 degrees
- moved C5 3.16 mm to (41.0, 62.0), turned to -90 degrees
- moved C7 2.50 mm to (54.5, 39.0)
- moved C2 1.50 mm to (47.5, 41.0), turned to -90 degrees
- moved C3 1.41 mm to (41.0, 49.0), turned to -90 degrees
- moved U1 1.14 mm to (63.4, 39.0)
- moved C1 1.00 mm to (41.0, 41.0), turned to -90 degrees
Routing:
- net Net-(R4-Pad1): track 0.00 -> 60.4 mm
- net Net-(R3-Pad1): track 0.00 -> 56.7 mm
- net Net-(C5-Pad1): track 0.00 -> 56.2 mm
- net Net-(C4-Pad1): track 0.00 -> 49.8 mm, vias 0 -> 1
- net Net-(R1-Pad1): track 0.00 -> 38.7 mm
- net Net-(R2-Pad1): track 0.00 -> 36.2 mm
- net Net-(C3-Pad1): track 0.00 -> 35.2 mm
- net Net-(C1-Pad1): track 0.00 -> 34.3 mm
- net VCC: track 0.00 -> 33.1 mm
- net step 3: track 0.00 -> 30.8 mm
- net step 2: track 0.00 -> 26.4 mm
- net step 4: track 0.00 -> 22.9 mm
- net out 1: track 0.00 -> 18.9 mm
- net out 3: track 0.00 -> 17.3 mm
- net step 1: track 0.00 -> 13.3 mm
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- added copper zone on B.Cu, net GND
- added copper zone on F.Cu, net GND
